File: V3sDevBoard/V3sDevBoard.kicad_pcb (KiCad board)
At the start: 4 copper layers, 100 x 85 mm, 191 parts, among them J1 JST_ETHERNET, J2 USB_C_Receptacle_USB2.0_16P, J3 USB_C_Receptacle_USB2.0_16P, J4 Micro_SD_Card_Det1, J5 LCD, J6 MIPI CSI, J7 JST_I2C, J8 AudioJack, J9 Conn_01x07_Pin, SW1 BUT6, SW2 BUT1, SW3 BUT2, SW4 BUT3, SW5 BUT4, SW6 BUT5, U1 Allwinner_V3s, U10 MPU-6050, U11 BME280, U12 USBLC6, U13 USBLC6, U14 USBLC6, U15 USBLC6, U16 USBLC6, U2 SY8089AAAC, U3 SY8089AAAC, U4 SY8089AAAC, U5 CH340C, U6 PT4103, U8 ESP32-WROOM-32, U9 Ai-Thinker-Ra-02, Y1 32K, Y2 24M

Commit message: update readme
Parts:
- removed JP6: vcc-rtc, Jumper:SolderJumper-2_P1.3mm_Bridged_RoundedPad1.0x1.5mm
Routing:
- net Net-(BT1-+): track 7.28 -> 4.05 mm
- net +3.3V: track 149.1 -> 148.0 mm, vias 41 -> 40
