File: V3sDevBoard/power.kicad_sch (KiCad schematic)
At the start: 45 parts, among them U2 SY8089AAAC, U3 SY8089AAAC, U4 SY8089AAAC, U6 PT4103

Commit message: update readme
Changed lines of the file:
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@@
 	(wire
 		(pts
-			(xy 121.92 49.53) (xy 113.03 49.53)
+			(xy 113.03 49.53) (xy 121.92 49.53)
 		)
 		(stroke
